File: PCB/Keyboard.kicad_pcb (KiCad board)
At the start: 2 copper layers, 404.8 x 140.5 mm, 163 parts, among them SW1 SW_Push, SW10 SW_Push, SW11 SW_Push, SW12 SW_Push, SW13 SW_Push, SW14 SW_Push, SW15 SW_Push, SW16 SW_Push, SW17 SW_Push, SW18 SW_Push, SW19 SW_Push, SW2 SW_Push, SW20 SW_Push, SW21 SW_Push, SW22 SW_Push, SW23 SW_Push, SW24 SW_Push, SW25 SW_Push, SW26 SW_Push, SW27 SW_Push, SW28 SW_Push, SW29 SW_Push, SW3 SW_Push, SW30 SW_Push, SW31 SW_Push, SW32 SW_Push, SW33 SW_Push, SW34 SW_Push, SW35 SW_Push, SW36 SW_Push, SW37 SW_Push, SW38 SW_Push, SW39 SW_Push, SW4 SW_Push, SW40 SW_Push, SW41 SW_Push, SW42 SW_Push, SW43 SW_Push, SW44 SW_Push, SW45 SW_Push, SW46 SW_Push, SW47 SW_Push, SW48 SW_Push, SW49 SW_Push, SW5 SW_Push, SW50 SW_Push, SW51 SW_Push, SW52 SW_Push, SW53 SW_Push, SW54 SW_Push, SW55 SW_Push, SW56 SW_Push, SW57 SW_Push, SW58 SW_Push, SW59 SW_Push, SW6 SW_Push, SW60 SW_Push, SW61 SW_Push, SW62 SW_Push, SW63 SW_Push, SW66 SW_Push, SW7 SW_Push, SW70 SW_Push, SW71 SW_Push, SW72 SW_Push, SW73 SW_Push, SW74 SW_Push, SW75 SW_Push, SW76 SW_Push, SW77 SW_Push, SW78 SW_Push, SW79 SW_Push, SW8 SW_Push, SW80 SW_Push, SW81 SW_Push, SW82 SW_Push, SW83 SW_Push, SW84 SW_Push, SW9 SW_Push

Commit message: Add files via upload
Connections:
- A1 pad TP5: unconnected-(A1-LED_OUT-PadTP5) -> LED
- D66 pad 1: unconnected-(D66-DOUT-Pad1) -> Net-(D66-DOUT)
- D66 pad 3: unconnected-(D66-DIN-Pad3) -> LED
- D67 pad 1: unconnected-(D67-DOUT-Pad1) -> Net-(D67-DOUT)
- D67 pad 3: unconnected-(D67-DIN-Pad3) -> Net-(D66-DOUT)
- D68 pad 1: unconnected-(D68-DOUT-Pad1) -> Net-(D68-DOUT)
- D68 pad 3: unconnected-(D68-DIN-Pad3) -> Net-(D67-DOUT)
- D69 pad 3: unconnected-(D69-DIN-Pad3) -> Net-(D68-DOUT)
Routing:
- net LED: track 0.00 -> 387.3 mm, vias 0 -> 4
- net Net-(D67-DOUT): track 0.00 -> 203.4 mm, vias 0 -> 4
- net Net-(D68-DOUT): track 0.00 -> 88.4 mm, vias 0 -> 4
- net Net-(D66-DOUT): track 0.00 -> 87.1 mm, vias 0 -> 2
- net Row 4: track 574.1 -> 572.6 mm

Commit message: Add files via upload
Connections:
- A1 pad 31: unconnected-(A1-GPIO26_ADC0-Pad31) -> LED
- A1 pad TP5: LED -> unconnected-(A1-LED_OUT-PadTP5)
Routing:
- net LED: track 387.3 -> 369.1 mm
Changed lines of the file:
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@@
 	(net 13 "C3")
 	(net 14 "C15")
-	(net 15 "unconnected-(A1-GPIO26_ADC0-Pad31)")
+	(net 15 "unconnected-(A1-LED_OUT-PadTP5)")
 	(net 16 "LED")
 	(net 17 "C7")
@@
 			(layers "F.Cu" "F.Mask")
 			(roundrect_rratio 0.5)
-			(net 15 "unconnected-(A1-GPIO26_ADC0-Pad31)")
+			(net 16 "LED")
 			(pinfunction "GPIO26_ADC0")
 			(pintype "bidirectional")
@@
 			(layers "F.Cu" "F.Mask" "F.Paste")
 			(roundrect_rratio 0.2)
-			(net 16 "LED")
+			(net 15 "unconnected-(A1-LED_OUT-PadTP5)")
 			(pinfunction "LED_OUT")
 			(pintype "output")
@@
 	)
 	(segment
+		(start 413.6875 72.7875)
+		(end 413.6875 69.5)
+		(width 0.2)
+		(layer "F.Cu")
+		(net 16)
+	)
+	(segment
 		(start 132 130.7)
 		(end 133.3 130.7)
@@
 	)
 	(segment
+		(start 414 73.1)
+		(end 413.6875 72.7875)
+		(width 0.2)
+		(layer "F.Cu")
+		(net 16)
+	)
+	(segment
 		(start 133.3 130.7)
 		(end 134.9 129.1)
@@
 	)
 	(segment
-		(start 427.4 62.3)
-		(end 427.4175 62.2825)
-		(width 0.2)
-		(layer "F.Cu")
-		(net 16)
-	)
-	(segment
 		(start 120.8125 127.08125)
 		(end 124.43125 130.7)
@@
 	)
 	(segment
-		(start 427.4175 62.2825)
-		(end 427.4175 57.31)
-		(width 0.2)
-		(layer "F.Cu")
-		(net 16)
-	)
-	(segment
 		(start 130.6 81.1)
 		(end 124.8 86.9)
@@
 	)
 	(via
-		(at 427.4 62.3)
+		(at 137.7 77.2)
 		(size 0.6)
 		(drill 0.3)
@@
 	)
 	(via
-		(at 137.7 77.2)
+		(at 414 73.1)
 		(size 0.6)
 		(drill 0.3)
@@
 	)
 	(segment
-		(start 124.8 118.3)
-		(end 124.8 117.7)
+		(start 414.799 75.1)
+		(end 412.699 77.2)
 		(width 0.2)
 		(layer "B.Cu")
@@
 	)
 	(segment
-		(start 124.8 117.7)
-		(end 124.8 114.4)
+		(start 124.8 118.3)
+		(end 124.8 117.7)
 		(width 0.2)
 		(layer "B.Cu")
@@
 	)
 	(segment
-		(start 414.799 77.2)
-		(end 427.4 64.599)
+		(start 414 73.1)
+		(end 414.799 73.899)
 		(width 0.2)
 		(layer "B.Cu")
@@
 	)
 	(segment
-		(start 427.4 64.599)
-		(end 427.4 62.3)
+		(start 124.8 117.7)
+		(end 124.8 114.4)
 		(width 0.2)
 		(layer "B.Cu")
@@
 	)
 	(segment
-		(start 137.7 77.2)
-		(end 414.799 77.2)
+		(start 412.699 77.2)
+		(end 137.7 77.2)
 		(width 0.2)
 		(layer "B.Cu")
@@
 		(width 0.2)
 		(layer "B.Cu")
+		(net 16)
+	)
+	(segment
+		(start 414.799 73.899)
+		(end 414.799 75.1)
+		(width 0.2)
+		(layer "B.Cu")
