File: PCB/Keyboard.kicad_sch (KiCad schematic)
At the start: 163 parts, among them SW1 SW_Push, SW10 SW_Push, SW11 SW_Push, SW12 SW_Push, SW13 SW_Push, SW14 SW_Push, SW15 SW_Push, SW16 SW_Push, SW17 SW_Push, SW18 SW_Push, SW19 SW_Push, SW2 SW_Push, SW20 SW_Push, SW21 SW_Push, SW22 SW_Push, SW23 SW_Push, SW24 SW_Push, SW25 SW_Push, SW26 SW_Push, SW27 SW_Push, SW28 SW_Push, SW29 SW_Push, SW3 SW_Push, SW30 SW_Push, SW31 SW_Push, SW32 SW_Push, SW33 SW_Push, SW34 SW_Push, SW35 SW_Push, SW36 SW_Push, SW37 SW_Push, SW38 SW_Push, SW39 SW_Push, SW4 SW_Push, SW40 SW_Push, SW41 SW_Push, SW42 SW_Push, SW43 SW_Push, SW44 SW_Push, SW45 SW_Push, SW46 SW_Push, SW47 SW_Push, SW48 SW_Push, SW49 SW_Push, SW5 SW_Push, SW50 SW_Push, SW51 SW_Push, SW52 SW_Push, SW53 SW_Push, SW54 SW_Push, SW55 SW_Push, SW56 SW_Push, SW57 SW_Push, SW58 SW_Push, SW59 SW_Push, SW6 SW_Push, SW60 SW_Push, SW61 SW_Push, SW62 SW_Push, SW63 SW_Push, SW66 SW_Push, SW7 SW_Push, SW70 SW_Push, SW71 SW_Push, SW72 SW_Push, SW73 SW_Push, SW74 SW_Push, SW75 SW_Push, SW76 SW_Push, SW77 SW_Push, SW78 SW_Push, SW79 SW_Push, SW8 SW_Push, SW80 SW_Push, SW81 SW_Push, SW82 SW_Push, SW83 SW_Push, SW84 SW_Push, SW9 SW_Push

Commit message: Add files via upload
Parts:
- SW14, SW44, SW46, SW57: footprint Button_Switch_Keyboard:SW_Cherry_MX_1.00u_PCB -> Button_Switch_Keyboard:SW_Cherry_MX_2.00u_PCB
- SW16, SW29: footprint Button_Switch_Keyboard:SW_Cherry_MX_1.00u_PCB -> Button_Switch_Keyboard:SW_Cherry_MX_1.50u_PCB
- SW43: footprint Button_Switch_Keyboard:SW_Cherry_MX_1.00u_PCB -> Button_Switch_Keyboard:SW_Cherry_MX_2.25u_PCB
- SW61, SW62, SW63: footprint Button_Switch_Keyboard:SW_Cherry_MX_1.00u_PCB -> Button_Switch_Keyboard:SW_Cherry_MX_1.25u_PCB
- SW66: footprint Button_Switch_Keyboard:SW_Cherry_MX_1.00u_PCB -> Button_Switch_Keyboard:SW_Cherry_MX_6.25u_PCB
Changed lines of the file:
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@@
 			)
 		)
-		(property "Footprint" "Button_Switch_Keyboard:SW_Cherry_MX_1.00u_PCB"
+		(property "Footprint" "Button_Switch_Keyboard:SW_Cherry_MX_2.00u_PCB"
 			(at 226.06 121.92 0)
 			(effects
@@
 			)
 		)
-		(property "Footprint" "Button_Switch_Keyboard:SW_Cherry_MX_1.00u_PCB"
+		(property "Footprint" "Button_Switch_Keyboard:SW_Cherry_MX_1.25u_PCB"
 			(at 55.88 147.32 0)
 			(effects
@@
 			)
 		)
-		(property "Footprint" "Button_Switch_Keyboard:SW_Cherry_MX_1.00u_PCB"
+		(property "Footprint" "Button_Switch_Keyboard:SW_Cherry_MX_2.00u_PCB"
 			(at 55.88 121.92 0)
 			(effects
@@
 			)
 		)
-		(property "Footprint" "Button_Switch_Keyboard:SW_Cherry_MX_1.00u_PCB"
+		(property "Footprint" "Button_Switch_Keyboard:SW_Cherry_MX_1.50u_PCB"
 			(at 55.88 71.12 0)
 			(effects
@@
 			)
 		)
-		(property "Footprint" "Button_Switch_Keyboard:SW_Cherry_MX_1.00u_PCB"
+		(property "Footprint" "Button_Switch_Keyboard:SW_Cherry_MX_2.25u_PCB"
 			(at 241.3 96.52 0)
 			(effects
@@
 			)
 		)
-		(property "Footprint" "Button_Switch_Keyboard:SW_Cherry_MX_1.00u_PCB"
+		(property "Footprint" "Button_Switch_Keyboard:SW_Cherry_MX_1.25u_PCB"
 			(at 86.36 147.32 0)
 			(effects
@@
 			)
 		)
-		(property "Footprint" "Button_Switch_Keyboard:SW_Cherry_MX_1.00u_PCB"
+		(property "Footprint" "Button_Switch_Keyboard:SW_Cherry_MX_1.25u_PCB"
 			(at 71.12 147.32 0)
 			(effects
@@
 			)
 		)
-		(property "Footprint" "Button_Switch_Keyboard:SW_Cherry_MX_1.00u_PCB"
+		(property "Footprint" "Button_Switch_Keyboard:SW_Cherry_MX_6.25u_PCB"
 			(at 133.35 147.32 0)
 			(effects
@@
 			)
 		)
-		(property "Footprint" "Button_Switch_Keyboard:SW_Cherry_MX_1.00u_PCB"
+		(property "Footprint" "Button_Switch_Keyboard:SW_Cherry_MX_1.50u_PCB"
 			(at 256.54 71.12 0)
 			(effects
@@
 			)
 		)
-		(property "Footprint" "Button_Switch_Keyboard:SW_Cherry_MX_1.00u_PCB"
+		(property "Footprint" "Button_Switch_Keyboard:SW_Cherry_MX_2.00u_PCB"
 			(at 256.54 45.72 0)
 			(effects
@@
 			)
 		)
-		(property "Footprint" "Button_Switch_Keyboard:SW_Cherry_MX_1.00u_PCB"
+		(property "Footprint" "Button_Switch_Keyboard:SW_Cherry_MX_2.00u_PCB"
 			(at 55.88 261.62 0)
 			(effects

Commit message: Add files via upload
Connections:
- net at D67.1 (DOUT): now also D68.3 (DIN)
- net at D67.3 (DIN): now also D66.1 (DOUT)
- net LED: now reaches D66.3 (DIN)
- net LED: now also A1.TP5 (LED_OUT)
- net at D68.1 (DOUT): now also D69.3 (DIN)
Changed lines of the file:
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@@
 	)
 	(junction
+		(at 201.93 176.53)
+		(diameter 0)
+		(color 0 0 0 0)
+	)
+	(junction
 		(at 106.68 58.42)
 		(diameter 0)
@@
 	)
 	(junction
-		(at 201.93 176.53)
-		(diameter 0)
-		(color 0 0 0 0)
-	)
-	(junction
 		(at 231.14 160.02)
 		(diameter 0)
@@
 	(wire
 		(pts
+			(xy 167.64 184.15) (xy 172.72 184.15)
+		)
+		(stroke
+			(width 0)
+			(type default)
+		)
+	)
+	(wire
+		(pts
 			(xy 60.96 274.32) (xy 93.98 274.32)
 		)
@@
 	(wire
 		(pts
+			(xy 130.81 184.15) (xy 132.08 184.15)
+		)
+		(stroke
+			(width 0)
+			(type default)
+		)
+	)
+	(wire
+		(pts
 			(xy 231.14 160.02) (xy 246.38 160.02)
 		)
@@
 	(wire
 		(pts
-			(xy 261.62 134.62) (xy 276.86 134.62)
+			(xy 201.93 194.31) (xy 201.93 191.77)
 		)
 		(stroke
@@
 	(wire
 		(pts
-			(xy 50.8 127) (xy 50.8 152.4)
+			(xy 261.62 134.62) (xy 276.86 134.62)
 		)
 		(stroke
@@
 	(wire
 		(pts
-			(xy 168.91 109.22) (xy 184.15 109.22)
+			(xy 50.8 127) (xy 50.8 152.4)
 		)
 		(stroke
@@
 	(wire
 		(pts
-			(xy 50.8 190.5) (xy 50.8 215.9)
+			(xy 168.91 109.22) (xy 184.15 109.22)
 		)
 		(stroke
@@
 	(wire
 		(pts
-			(xy 50.8 215.9) (xy 50.8 241.3)
+			(xy 50.8 190.5) (xy 50.8 215.9)
 		)
 		(stroke
@@
 	(wire
 		(pts
-			(xy 201.93 193.04) (xy 201.93 191.77)
+			(xy 50.8 215.9) (xy 50.8 241.3)
 		)
 		(stroke
@@
 	(wire
 		(pts
-			(xy 201.93 175.26) (xy 201.93 176.53)
-		)
-		(stroke
-			(width 0)
-			(type default)
-		)
-	)
-	(wire
-		(pts
 			(xy 96.52 76.2) (xy 96.52 101.6)
 		)
@@
 	(wire
 		(pts
+			(xy 201.93 173.99) (xy 201.93 176.53)
+		)
+		(stroke
+			(width 0)
+			(type default)
+		)
+	)
+	(wire
+		(pts
 			(xy 138.43 109.22) (xy 153.67 109.22)
 		)
@@
 	(wire
 		(pts
+			(xy 147.32 184.15) (xy 152.4 184.15)
+		)
+		(stroke
+			(width 0)
+			(type default)
+		)
+	)
+	(wire
+		(pts
 			(xy 81.28 50.8) (xy 81.28 76.2)
 		)
@@
 	(wire
 		(pts
+			(xy 187.96 184.15) (xy 194.31 184.15)
+		)
+		(stroke
+			(width 0)
+			(type default)
+		)
+	)
+	(wire
+		(pts
 			(xy 121.92 109.22) (xy 138.43 109.22)
 		)
@@
 		)
 	)
+	(global_label "LED"
+		(shape input)
+		(at 130.81 184.15 180)
+		(fields_autoplaced yes)
+		(effects
+			(font
+				(size 1.27 1.27)
+			)
+			(justify right)
+		)
+		(property "Intersheetrefs" "${INTERSHEET_REFS}"
+			(at 124.3777 184.15 0)
+			(effects
+				(font
+					(size 1.27 1.27)
+				)
+				(justify right)
+				(hide yes)
+			)
+		)
+	)
 	(global_label "Row 4x"
 		(shape input)
@@
 		)
 	)
+	(global_label "LED"
+		(shape input)
+		(at 375.92 62.23 0)
+		(fields_autoplaced yes)
+		(effects
+			(font
+				(size 1.27 1.27)
+			)
+			(justify left)
+		)
+		(property "Intersheetrefs" "${INTERSHEET_REFS}"
+			(at 382.3523 62.23 0)
+			(effects
+				(font
+					(size 1.27 1.27)
+				)
+				(justify left)
+				(hide yes)
+			)
+		)
+	)
 	(global_label "Row 3"
 		(shape input)
@@
 	(symbol
 		(lib_id "power:+5V")
-		(at 201.93 175.26 0)
+		(at 201.93 173.99 0)
 		(unit 1)
 		(exclude_from_sim no)
@@
 		(fields_autoplaced yes)
 		(property "Reference" "#PWR03"
-			(at 201.93 179.07 0)
+			(at 201.93 177.8 0)
 			(effects
 				(font
@@
 		)
 		(property "Value" "+5V"
-			(at 201.93 170.18 0)
+			(at 201.93 168.91 0)
 			(effects
 				(font
@@
 		)
 		(property "Footprint" ""
-			(at 201.93 175.26 0)
+			(at 201.93 173.99 0)
 			(effects
 				(font
@@
 		)
 		(property "Datasheet" ""
-			(at 201.93 175.26 0)
+			(at 201.93 173.99 0)
 			(effects
 				(font
@@
 		)
 		(property "Description" "Power symbol creates a global label with name \"+5V\""
-			(at 201.93 175.26 0)
+			(at 201.93 173.99 0)
 			(effects
 				(font
@@
 	(symbol
 		(lib_id "power:GND")
-		(at 201.93 193.04 0)
+		(at 201.93 194.31 0)
 		(unit 1)
 		(exclude_from_sim no)
@@
 		(fields_autoplaced yes)
 		(property "Reference" "#PWR01"
-			(at 201.93 199.39 0)
+			(at 201.93 200.66 0)
 			(effects
 				(font
@@
 		)
 		(property "Value" "GND"
-			(at 201.93 198.12 0)
+			(at 201.93 199.39 0)
 			(effects
 				(font
@@
 		)
 		(property "Footprint" ""
-			(at 201.93 193.04 0)
+			(at 201.93 194.31 0)
 			(effects
 				(font
@@
 		)
 		(property "Datasheet" ""
-			(at 201.93 193.04 0)
+			(at 201.93 194.31 0)
 			(effects
 				(font
@@
 		)
 		(property "Description" "Power symbol creates a global label with name \"GND\" , ground"
-			(at 201.93 193.04 0)
+			(at 201.93 194.31 0)
 			(effects
 				(font

Commit message: Add files via upload
Connections:
- net LED: now also A1.31 (GPIO26_ADC0); no longer A1.TP5 (LED_OUT)
